File: SC440_Preamp.kicad_pcb (KiCad board)
At the start: 2 copper layers, 30 x 35 mm, 29 parts, among them J1 JST-XH 1x04 TO DIGITAL BOARD, J2 ANALOG BOARD, U1 OPA1678IDR

Commit message: this project won't really help
Parts:
- TP1, TP2, TP3, TP4, TP5: footprint TestPoint:TestPoint_THTPad_1.0x1.0mm_Drill0.5mm -> TestPoint:TestPoint_THTPad_D1.0mm_Drill0.5mm
Connections:
- REF** pad 1: (no net) -> GND (x2)
- REF** pad 2: (no net) -> GND (x2)
Routing:
- net /VREF_RAW: track 14.4 -> 16.0 mm
Other:
- board text added: "PRE AMP OUT"
- board text removed: "PREAMP"
